File: MorphWatch-Hardware/MorphWatch-STM32.kicad_pcb (KiCad board)
At the start: 4 copper layers, 33.8 x 46 mm, 64 parts, among them IC1 ME6211C33M5G-N, J1 USB, J2 Conn_01x24, J3 Conn_01x04, J4 Conn_01x02, J5 Conn_01x05, M1 Motor_DC_ALT, Q1 CJ2301_S1, Q2 DMN3042L, Q3 S8050, U1 TP4054, U2 STM32L476RGTx, U3 JDY-08, U4 MPU-6050, Y1 Crystal_GND24

Commit message: Made changes to satisfy DRC
Parts:
- moved TP1 0.58 mm to (139.5, 94.7)
- moved C7 0.47 mm to (130.1, 97.5)
- moved R8 0.32 mm to (143.0, 78.3)
- moved R9 0.25 mm to (143.0, 77.2)
- moved R1 0.19 mm to (131.0, 91.1)
Routing:
- net GND: track 121.6 -> 124.9 mm, vias 28 -> 27
- net imuSDA: track 11.1 -> 10.0 mm
- net RESE: track 19.4 -> 20.1 mm
- net Net-(C4-Pad1): track 19.5 -> 20.1 mm
- net BATT_STAT: track 12.3 -> 11.8 mm
- net +3V3: vias 18 -> 17
Other:
- board text added: "+"
- board text added: "-"
- board text added: "GND"
- board text added: "RST"
- board text added: "SWD"
- board text added: "swc"
- board text added: "swo"
